File: Charj_Smol.kicad_sch (KiCad schematic)
At the start: 18 parts, among them J1 Battery Connector, Q1 PMN30XPEX, U1 MCP73831-2-OT, U2 LC709203FXE-05MH

Commit message: Silkscreen tidying; still Rev C
Parts:
- PADS1, PADS2, PADS3: now left out of the parts list
Changed lines of the file:
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@@
   )
   (symbol (lib_id "Connector_Generic:Conn_01x06") (at 251.46 121.92 180) (unit 1)
-    (in_bom yes) (on_board yes) (fields_autoplaced)
+    (in_bom no) (on_board yes) (fields_autoplaced)
     (property "Reference" "PADS1" (id 0) (at 249.428 119.7415 0)
       (effects (font (size 1.27 1.27)) (justify left))
@@
   )
   (symbol (lib_id "Connector_Generic:Conn_01x01") (at 251.46 139.7 0) (mirror y) (unit 1)
-    (in_bom yes) (on_board yes) (fields_autoplaced)
+    (in_bom no) (on_board yes) (fields_autoplaced)
     (property "Reference" "PADS3" (id 0) (at 249.4281 138.7915 0)
       (effects (font (size 1.27 1.27)) (justify left))
@@
   )
   (symbol (lib_id "Connector_Generic:Conn_01x06") (at 251.46 101.6 180) (unit 1)
-    (in_bom yes) (on_board yes)
+    (in_bom no) (on_board yes)
     (property "Reference" "PADS2" (id 0) (at 251.46 85.09 0))
     (property "Value" "Underside Pads" (id 1) (at 251.46 88.9 0))
